Commit message: Following changes are added: 1. Introduced 4 wheels(Link names: left_wheel_1, left_wheel_2, right_wheel_1, right_wheel_2) 2. Added Camera. 3. Added LIDAR. Known Issue: Wheel colors are not able to change, debug it further

File: four_wheel_robot/catkin_ws/src/my_robot/urdf/my_robot.xacro (robot description, xacro)
@@ -7,5 +7,5 @@
   </joint>
   <link name='chassis'>
-    <pose>0 0 0.1 0 0 0</pose>
+    <pose>0 0 0.3 0 0 0</pose>
     <inertial>
       <mass value="15.0"/>
@@ -20,5 +20,5 @@
       <origin xyz="0 0 0" rpy=" 0 0 0"/>
       <geometry>
-        <box size=".4 .2 .1"/>
+        <box size=".6 .24 .1"/>
       </geometry>
     </collision>
@@ -26,5 +26,5 @@
       <origin xyz="0 0 0" rpy=" 0 0 0"/>
       <geometry>
-        <box size=".4 .2 .1"/>
+        <box size=".6 .24 .1"/>
       </geometry>
     </visual>
@@ -54,3 +54,196 @@
     </visual>
   </link>
+  <link name ="left_wheel_1">
+   <inertial>
+     <mass value="5.0"/>
+     <origin xyz="0 0 0" rpy="0 1.5707 1.5707"/>
+     <inertia
+          ixx="0.1" ixy="0" ixz="0"
+          iyy="0.1" iyz="0"
+          izz="0.1"/>
+    </inertial>
+   <collision name="left_wheel_collision_1">
+     <origin xyz="0 0 0" rpy="0 1.5707 1.5707"/>
+     <geometry>
+       <cylinder radius="0.1" length="0.05"/>
+     </geometry>
+   </collision>
+   <visual name="left_wheel_visual_1">
+     <origin xyz="0 0 0" rpy="0 1.5707 1.5707"/>
+     <geometry>
+       <cylinder radius="0.1" length="0.05"/>
+     </geometry>
+   </visual>
+  </link>
+  <joint type="continuous" name="left_wheel_hinge_1">
+    <origin xyz="0.15 0.15 0" rpy="0 0 0"/>
+    <child link="left_wheel_1"/>
+    <parent link="chassis"/>
+    <axis xyz="0 1 0" rpy="0 0 0"/>
+    <limit effort="10000" velocity="1000"/>
+    <dynamics damping="1.0" friction="1.0"/>
+  </joint>
+  <link name ="left_wheel_2">
+   <inertial>
+     <mass value="5.0"/>
+     <origin xyz="0 0 0" rpy="0 1.5707 1.5707"/>
+     <inertia
+          ixx="0.1" ixy="0" ixz="0"
+          iyy="0.1" iyz="0"
+          izz="0.1"/>
+    </inertial>
+   <collision name="left_wheel_collision_2">
+     <origin xyz="0 0 0" rpy="0 1.5707 1.5707"/>
+     <geometry>
+       <cylinder radius="0.1" length="0.05"/>
+     </geometry>
+   </collision>
+   <visual name="left_wheel_visual_2">
+     <origin xyz="0 0 0" rpy="0 1.5707 1.5707"/>
+     <geometry>
+       <cylinder radius="0.1" length="0.05"/>
+     </geometry>
+   </visual>
+  </link>
+  <joint type="continuous" name="left_wheel_hinge_2">
+    <origin xyz="-0.15 0.15 0" rpy="0 0 0"/>
+    <child link="left_wheel_2"/>
+    <parent link="chassis"/>
+    <axis xyz="0 1 0" rpy="0 0 0"/>
+    <limit effort="10000" velocity="1000"/>
+    <dynamics damping="1.0" friction="1.0"/>
+  </joint>
+  <link name ="right_wheel_1">
+   <inertial>
+     <mass value="5.0"/>
+     <origin xyz="0 0 0" rpy="0 1.5707 1.5707"/>
+     <inertia
+          ixx="0.1" ixy="0" ixz="0"
+          iyy="0.1" iyz="0"
+          izz="0.1"/>
+    </inertial>
+   <collision name="right_wheel_collision_1">
+     <origin xyz="0 0 0" rpy="0 1.5707 1.5707"/>
+     <geometry>
+       <cylinder radius="0.1" length="0.05"/>
+     </geometry>
+   </collision>
+   <visual name="right_wheel_visual_1">
+     <origin xyz="0 0 0" rpy="0 1.5707 1.5707"/>
+     <geometry>
+       <cylinder radius="0.1" length="0.05"/>
+     </geometry>
+   </visual>
+  </link>
+  <joint type="continuous" name="right_wheel_hinge_1">
+    <origin xyz="0.15 -0.15 0" rpy="0 0 0"/>
+    <child link="right_wheel_1"/>
+    <parent link="chassis"/>
+    <axis xyz="0 1 0" rpy="0 0 0"/>
+    <limit effort="10000" velocity="1000"/>
+    <dynamics damping="1.0" friction="1.0"/>
+  </joint>
+  <link name ="right_wheel_2">
+   <inertial>
+     <mass value="5.0"/>
+     <origin xyz="0 0 0" rpy="0 1.5707 1.5707"/>
+     <inertia
+          ixx="0.1" ixy="0" ixz="0"
+          iyy="0.1" iyz="0"
+          izz="0.1"/>
+    </inertial>
+   <collision name="right_wheel_collision_2">
+     <origin xyz="0 0 0" rpy="0 1.5707 1.5707"/>
+     <geometry>
+       <cylinder radius="0.1" length="0.05"/>
+     </geometry>
+   </collision>
+   <visual name="right_wheel_visual_2">
+     <origin xyz="0 0 0" rpy="0 1.5707 1.5707"/>
+     <geometry>
+       <cylinder radius="0.1" length="0.05"/>
+     </geometry>
+     <material name="black" />
+   </visual>
+  </link>
+  <joint type="continuous" name="right_wheel_hinge_2">
+    <origin xyz="-0.15 -0.15 0" rpy="0 0 0"/>
+    <child link="right_wheel_2"/>
+    <parent link="chassis"/>
+    <axis xyz="0 1 0" rpy="0 0 0"/>
+    <limit effort="10000" velocity="1000"/>
+    <dynamics damping="1.0" friction="1.0"/>
+  </joint>
+  <link name = "camera">
+    <inertial>
+      <mass value="0.1" />
+      <origin xyz="0.05 0.05 0.05" rpy="0 0 0" />
+      <inertia ixx="0.0000001" ixy="0" ixz="0" iyy="0.0000001" iyz="0" izz="0.0000001" />
+    </inertial>
+    <collision>
+      <origin xyz="0 0 0" rpy="0 0 0"/>
+      <geometry>
+        <box size="0.05 0.05 0.05"/>
+      </geometry>
+    </collision>
+    <visual>
+      <origin xyz="0 0 0" rpy="0 0 0"/>
+      <geometry>
+        <box size="0.05 0.05 0.05"/>
+      </geometry>
+    </visual>
+  </link>
+ <joint name="camera_joint" type="fixed">
+            <axis xyz="0 1 0" />
+            <origin xyz="0.3 0 0" rpy="0 0 0"/>
+            <parent link="chassis"/>
+            <child link="camera"/>
+    </joint>
+ <link name="hokuyo">
+    <collision name='hokuyo_collision'>
+      <origin xyz="0 0 0" rpy="0 0 0"/>
+      <geometry>
+        <box size="0.1 0.1 0.1"/>
+      </geometry>
+    </collision>
+    <visual>
+      <origin xyz="0 0 0" rpy="0 0 0"/>
+      <geometry>
+        <mesh filename="package://my_robot/meshes/hokuyo.dae"/>
+      </geometry>
+    </visual>
+    <inertial>
+      <mass value="1e-5"/>
+      <origin xyz="0.0 0 0" rpy="0 0 0"/>
+      <inertia
+          ixx="1e-6" ixy="0" ixz="0"
+          iyy="1e-6" iyz="0"
+          izz="1e-6"
+      />
+    </inertial>
+  </link>
+  <joint type="fixed" name="hokuyo_joint">
+    <origin xyz="0.15 0 0.1" rpy="0 0 0"/>
+    <child link="hokuyo"/>
+    <parent link="chassis"/>
+    <axis xyz="0 1 0" rpy="0 0 0"/>
+  </joint>
+<gazebo reference="chassis">
+    <material>Gazebo/Blue</material>
+</gazebo>
+<gazebo reference="left_wheel_1">
+    <material>Gazebo/Green</material>
+</gazebo>
+<gazebo reference="left_wheel_2">
+    <material>Gazebo/Green</material>
+</gazebo>
+<gazebo reference="right_wheel_1">
+    <material>Gazebo/Green</material>
+</gazebo>
+<gazebo reference="right_wheel_2">
+    <material>Gazebo/Green</material>
+</gazebo>
+<gazebo reference="camera">
+    <material>Gazebo/Red</material>
+</gazebo>
 </robot>
