Commit message: Fixing as per review comments

File: go_chase_it/my_robot/urdf/my_robot.xacro (robot description, xacro)
@@ -1,4 +1,4 @@
 <robot name="my_robot" xmlns:xacro="http://www.ros.org/wiki/xacro">
- <xacro:include filename="$(find my_robot)/urdf/my_robot.gazebo" />
+<xacro:include filename="$(find my_robot)/urdf/my_robot.gazebo" />
   <link name="robot_footprint"></link>
   <joint name="robot_footprint_joint" type="fixed">
@@ -8,5 +8,5 @@
   </joint>
   <link name='chassis'>
-    <pose>0 0 0.1 0 0 0</pose>
+    <pose>0 0 0.3 0 0 0</pose>
     <inertial>
       <mass value="15.0"/>
@@ -21,5 +21,5 @@
       <origin xyz="0 0 0" rpy=" 0 0 0"/>
       <geometry>
-        <box size=".4 .2 .1"/>
+        <box size=".6 .24 .1"/>
       </geometry>
     </collision>
@@ -27,5 +27,5 @@
       <origin xyz="0 0 0" rpy=" 0 0 0"/>
       <geometry>
-        <box size=".4 .2 .1"/>
+        <box size=".6 .24 .1"/>
       </geometry>
     </visual>
@@ -136,8 +136,8 @@
  <joint name="camera_joint" type="fixed">
             <axis xyz="0 1 0" />
-            <origin xyz="0.2 0 0" rpy="0 0 0"/>
+            <origin xyz="0.3 0 0" rpy="0 0 0"/>
             <parent link="chassis"/>
             <child link="camera"/>
-    </joint>
+ </joint>
  <link name="hokuyo">
     <collision name='hokuyo_collision'>
@@ -170,14 +170,14 @@
   </joint>
 <gazebo reference="chassis">
-    <material>Gazebo/Blue</material>
+    <material>Gazebo/Yellow</material>
 </gazebo>
 <gazebo reference="left_wheel">
+    <material>Gazebo/Purple</material>
+</gazebo>
+<gazebo reference="right_wheel">
+    <material>Gazebo/Purple</material>
+</gazebo>
+<gazebo reference="camera">
     <material>Gazebo/Green</material>
 </gazebo>
-<gazebo reference="right_wheel">
-    <material>Gazebo/Green</material>
-</gazebo>
-<gazebo reference="camera">
-    <material>Gazebo/Red</material>
-</gazebo>
 </robot>

Commit message: Changed intertia, radius of the wwheel to 0.12 radius, origin of the wheel to -0.05

File: go_chase_it/my_robot/urdf/my_robot.xacro (robot description, xacro)
@@ -13,7 +13,7 @@
       <origin xyz="0.0 0 0" rpy=" 0 0 0"/>
       <inertia
-          ixx="0.1" ixy="0" ixz="0"
-          iyy="0.1" iyz="0"
-          izz="0.1"
+          ixx="0.08425" ixy="0" ixz="0"
+          iyy="0.318625" iyz="0"
+          izz="0.390625"
       />
     </inertial>
@@ -31,11 +31,11 @@
     </visual>
     <collision name='back_caster_collision'>
-      <origin xyz="-0.15 0 -0.05" rpy=" 0 0 0"/>
+      <origin xyz="-0.18 0 -0.06" rpy=" 0 0 0"/>
       <geometry>
-        <sphere radius="0.0499"/>
+        <sphere radius="0.05"/>
       </geometry>
     </collision>
     <visual name='back_caster_visual'>
-      <origin xyz="-0.15 0 -0.05" rpy=" 0 0 0"/>
+      <origin xyz="-0.18 0 -0.06" rpy=" 0 0 0"/>
       <geometry>
         <sphere radius="0.05"/>
@@ -43,11 +43,11 @@
     </visual>
     <collision name='front_caster_collision'>
-      <origin xyz="0.15 0 -0.05" rpy=" 0 0 0"/>
+      <origin xyz="0.18 0 -0.06" rpy=" 0 0 0"/>
       <geometry>
-        <sphere radius="0.0499"/>
+        <sphere radius="0.05"/>
       </geometry>
     </collision>
     <visual name='front_caster_visual'>
-      <origin xyz="0.15 0 -0.05" rpy=" 0 0 0"/>
+      <origin xyz="0.18 0 -0.06" rpy=" 0 0 0"/>
       <geometry>
         <sphere radius="0.05"/>
@@ -60,23 +60,23 @@
      <origin xyz="0 0 0" rpy="0 1.5707 1.5707"/>
      <inertia
-          ixx="0.1" ixy="0" ixz="0"
-          iyy="0.1" iyz="0"
-          izz="0.1"/>
+          ixx="0.013541666" ixy="0" ixz="0"
+          iyy="0.013541666" iyz="0"
+          izz="0.025"/>
     </inertial>
    <collision name="left_wheel_collision">
-     <origin xyz="0 0 0" rpy="0 1.5707 1.5707"/>
+     <origin xyz="-0.05 0 0" rpy="0 1.5707 1.5707"/>
      <geometry>
-       <cylinder radius="0.1" length="0.05"/>
+       <cylinder radius="0.12" length="0.05"/>
      </geometry>
    </collision>
    <visual name="left_wheel_visual">
-     <origin xyz="0 0 0" rpy="0 1.5707 1.5707"/>
+     <origin xyz="-0.05 0 0" rpy="0 1.5707 1.5707"/>
      <geometry>
-       <cylinder radius="0.1" length="0.05"/>
+       <cylinder radius="0.12" length="0.05"/>
      </geometry>
    </visual>
   </link>
   <joint type="continuous" name="left_wheel_hinge">
-    <origin xyz="0 0.15 0" rpy="0 0 0"/>
+    <origin xyz="-0.05 0.15 0" rpy="0 0 0"/>
     <child link="left_wheel"/>
     <parent link="chassis"/>
@@ -90,23 +90,23 @@
      <origin xyz="0 0 0" rpy="0 1.5707 1.5707"/>
      <inertia
-          ixx="0.1" ixy="0" ixz="0"
-          iyy="0.1" iyz="0"
-          izz="0.1"/>
+          ixx="0.013541666" ixy="0" ixz="0"
+          iyy="0.013541666" iyz="0"
+          izz="0.025"/>
     </inertial>
    <collision name="right_wheel_collision">
-     <origin xyz="0 0 0" rpy="0 1.5707 1.5707"/>
+     <origin xyz="-0.05 0 0" rpy="0 1.5707 1.5707"/>
      <geometry>
-       <cylinder radius="0.1" length="0.05"/>
+       <cylinder radius="0.12" length="0.05"/>
      </geometry>
    </collision>
    <visual name="right_wheel_visual">
-     <origin xyz="0 0 0" rpy="0 1.5707 1.5707"/>
+     <origin xyz="-0.05 0 0" rpy="0 1.5707 1.5707"/>
      <geometry>
-       <cylinder radius="0.1" length="0.05"/>
+       <cylinder radius="0.12" length="0.05"/>
      </geometry>
    </visual>
   </link>
   <joint type="continuous" name="right_wheel_hinge">
-    <origin xyz="0 -0.15 0" rpy="0 0 0"/>
+    <origin xyz="-0.05 -0.15 0" rpy="0 0 0"/>
     <child link="right_wheel"/>
     <parent link="chassis"/>

Commit message: Adding back_caster

File: go_chase_it/my_robot/urdf/my_robot.xacro (robot description, xacro)
@@ -8,12 +8,12 @@
   </joint>
   <link name='chassis'>
-    <pose>0 0 0.3 0 0 0</pose>
+    <pose>0 0 0.1 0 0 0</pose>
     <inertial>
       <mass value="15.0"/>
       <origin xyz="0.0 0 0" rpy=" 0 0 0"/>
       <inertia
-          ixx="0.08425" ixy="0" ixz="0"
-          iyy="0.318625" iyz="0"
-          izz="0.390625"
+          ixx="0.1" ixy="0" ixz="0"
+          iyy="0.1" iyz="0"
+          izz="0.1"
       />
     </inertial>
@@ -31,5 +31,5 @@
     </visual>
     <collision name='back_caster_collision'>
-      <origin xyz="-0.18 0 -0.06" rpy=" 0 0 0"/>
+      <origin xyz="-0.35 0 -0.05" rpy=" 0 0 0"/>
       <geometry>
         <sphere radius="0.05"/>
@@ -37,5 +37,5 @@
     </collision>
     <visual name='back_caster_visual'>
-      <origin xyz="-0.18 0 -0.06" rpy=" 0 0 0"/>
+      <origin xyz="-0.25 0 -0.05" rpy=" 0 0 0"/>
       <geometry>
         <sphere radius="0.05"/>
@@ -43,5 +43,5 @@
     </visual>
     <collision name='front_caster_collision'>
-      <origin xyz="0.18 0 -0.06" rpy=" 0 0 0"/>
+      <origin xyz="0.35 0 -0.05" rpy=" 0 0 0"/>
       <geometry>
         <sphere radius="0.05"/>
@@ -49,5 +49,5 @@
     </collision>
     <visual name='front_caster_visual'>
-      <origin xyz="0.18 0 -0.06" rpy=" 0 0 0"/>
+      <origin xyz="0.20 0 -0.05" rpy=" 0 0 0"/>
       <geometry>
         <sphere radius="0.05"/>
@@ -60,10 +60,10 @@
      <origin xyz="0 0 0" rpy="0 1.5707 1.5707"/>
      <inertia
-          ixx="0.013541666" ixy="0" ixz="0"
-          iyy="0.013541666" iyz="0"
-          izz="0.025"/>
+          ixx="0.1" ixy="0" ixz="0"
+          iyy="0.1" iyz="0"
+          izz="0.1"/>
     </inertial>
    <collision name="left_wheel_collision">
-     <origin xyz="-0.05 0 0" rpy="0 1.5707 1.5707"/>
+     <origin xyz="0 0 0" rpy="0 1.5707 1.5707"/>
      <geometry>
        <cylinder radius="0.12" length="0.05"/>
@@ -71,5 +71,5 @@
    </collision>
    <visual name="left_wheel_visual">
-     <origin xyz="-0.05 0 0" rpy="0 1.5707 1.5707"/>
+     <origin xyz="0 0 0" rpy="0 1.5707 1.5707"/>
      <geometry>
        <cylinder radius="0.12" length="0.05"/>
@@ -83,5 +83,5 @@
     <axis xyz="0 1 0" rpy="0 0 0"/>
     <limit effort="10000" velocity="1000"/>
-    <dynamics damping="1.0" friction="1.0"/>
+    <joint_properties damping="1.0" friction="1.0"/>
   </joint>
   <link name ="right_wheel">
@@ -90,10 +90,10 @@
      <origin xyz="0 0 0" rpy="0 1.5707 1.5707"/>
      <inertia
-          ixx="0.013541666" ixy="0" ixz="0"
-          iyy="0.013541666" iyz="0"
-          izz="0.025"/>
+          ixx="0.1" ixy="0" ixz="0"
+          iyy="0.1" iyz="0"
+          izz="0.1"/>
     </inertial>
    <collision name="right_wheel_collision">
-     <origin xyz="-0.05 0 0" rpy="0 1.5707 1.5707"/>
+     <origin xyz="0 0 0" rpy="0 1.5707 1.5707"/>
      <geometry>
        <cylinder radius="0.12" length="0.05"/>
@@ -101,5 +101,5 @@
    </collision>
    <visual name="right_wheel_visual">
-     <origin xyz="-0.05 0 0" rpy="0 1.5707 1.5707"/>
+     <origin xyz="0 0 0" rpy="0 1.5707 1.5707"/>
      <geometry>
        <cylinder radius="0.12" length="0.05"/>
@@ -113,5 +113,5 @@
     <axis xyz="0 1 0" rpy="0 0 0"/>
     <limit effort="10000" velocity="1000"/>
-    <dynamics damping="1.0" friction="1.0"/>
+    <joint_properties damping="1.0" friction="1.0"/>
   </joint>
   <link name = "camera">

Commit message: Changed the Pose to make more stable

File: go_chase_it/my_robot/urdf/my_robot.xacro (robot description, xacro)
@@ -11,13 +11,13 @@
     <inertial>
       <mass value="15.0"/>
-      <origin xyz="0.0 0 0" rpy=" 0 0 0"/>
+      <origin xyz="0 0 0" rpy=" 0 -0.05 0"/>
       <inertia
-          ixx="0.1" ixy="0" ixz="0"
-          iyy="0.1" iyz="0"
-          izz="0.1"
+          ixx="0.166667" ixy="0" ixz="0"
+          iyy="0.166667" iyz="0"
+          izz="0.166667"
       />
     </inertial>
     <collision name='collision'>
-      <origin xyz="0 0 0" rpy=" 0 0 0"/>
+      <origin xyz="0 0 0" rpy=" 0 -0.05 0"/>
       <geometry>
         <box size=".6 .24 .1"/>
@@ -25,5 +25,5 @@
     </collision>
     <visual name='chassis_visual'>
-      <origin xyz="0 0 0" rpy=" 0 0 0"/>
+      <origin xyz="0 0 0" rpy=" 0 -0.05 0"/>
       <geometry>
         <box size=".6 .24 .1"/>
@@ -31,5 +31,5 @@
     </visual>
     <collision name='back_caster_collision'>
-      <origin xyz="-0.35 0 -0.05" rpy=" 0 0 0"/>
+      <origin xyz="-0.23 0 -0.07" rpy=" 0 0 0"/>
       <geometry>
         <sphere radius="0.05"/>
@@ -37,5 +37,5 @@
     </collision>
     <visual name='back_caster_visual'>
-      <origin xyz="-0.25 0 -0.05" rpy=" 0 0 0"/>
+      <origin xyz="-0.23 0 -0.07" rpy=" 0 0 0"/>
       <geometry>
         <sphere radius="0.05"/>
@@ -43,5 +43,5 @@
     </visual>
     <collision name='front_caster_collision'>
-      <origin xyz="0.35 0 -0.05" rpy=" 0 0 0"/>
+      <origin xyz="0.23 0 -0.07" rpy=" 0 0 0"/>
       <geometry>
         <sphere radius="0.05"/>
@@ -49,5 +49,5 @@
     </collision>
     <visual name='front_caster_visual'>
-      <origin xyz="0.20 0 -0.05" rpy=" 0 0 0"/>
+      <origin xyz="0.23 0 -0.07" rpy=" 0 0 0"/>
       <geometry>
         <sphere radius="0.05"/>
@@ -60,7 +60,7 @@
      <origin xyz="0 0 0" rpy="0 1.5707 1.5707"/>
      <inertia
-          ixx="0.1" ixy="0" ixz="0"
-          iyy="0.1" iyz="0"
-          izz="0.1"/>
+          ixx="0.166667" ixy="0" ixz="0"
+          iyy="0.166667" iyz="0"
+          izz="0.166667"/>
     </inertial>
    <collision name="left_wheel_collision">
@@ -90,7 +90,7 @@
      <origin xyz="0 0 0" rpy="0 1.5707 1.5707"/>
      <inertia
-          ixx="0.1" ixy="0" ixz="0"
-          iyy="0.1" iyz="0"
-          izz="0.1"/>
+          ixx="0.166667" ixy="0" ixz="0"
+          iyy="0.166667" iyz="0"
+          izz="0.166667"/>
     </inertial>
    <collision name="right_wheel_collision">
